Commit message: Adjusted direction of robot coordinates, joints zero (home) position, and motion range. TODO: Get geometric accurate position of home

File: galil_description/urdf/galil.xacro (robot description, xacro)
@@ -5,5 +5,5 @@
     <link name="base_link">
       <visual>
-        <origin xyz="0 0 0" rpy="0 0 0"/>
+        <origin xyz="0 0 -0.025" rpy="0 0 ${-pi/2}"/>
         <geometry>
           <mesh filename="package://galil_description/meshes/base_link.stl"/>
@@ -12,14 +12,7 @@
       </visual>
     </link>
-    <link name="needle_link">
-      <visual>
-        <geometry>
-          <mesh filename="package://galil_description/meshes/needle_link.stl"/>
-        </geometry>
-        <material name="silver"/>
-      </visual>
-    </link>
     <link name="vertical_link">
       <visual>
+        <origin xyz="0 0 0" rpy="0 0 ${-pi/2}"/>
         <geometry>
           <mesh filename="package://galil_description/meshes/vertical_link.stl"/>
@@ -30,4 +23,5 @@
     <link name="horizontal_link">
       <visual>
+        <origin xyz="0 0 0" rpy="0 0 ${-pi/2}"/>
         <geometry>
           <mesh filename="package://galil_description/meshes/horizontal_link.stl"/>
@@ -36,10 +30,19 @@
       </visual>
     </link>
-    <joint name="insertion_joint" type="prismatic">
+    <link name="needle_link">
+      <visual>
+        <origin xyz="0 0 0" rpy="0 0 ${-pi/2}"/>
+        <geometry>
+          <mesh filename="package://galil_description/meshes/needle_link.stl"/>
+        </geometry>
+        <material name="silver"/>
+      </visual>
+    </link>
+    <joint name="vertical_joint" type="prismatic">
       <origin xyz="0 0 0" rpy="0 0 0"/>
-      <parent link="horizontal_link"/>
-      <child link="needle_link"/>
-      <axis xyz="-1.0 0.0 0.0"/>
-      <limit upper="0.1" lower="0.0" effort="100" velocity="100"/>
+      <parent link="base_link"/>
+      <child link="vertical_link"/>
+      <axis xyz="0.0 0.0 1.0"/>
+      <limit upper="0.025" lower="-0.025" effort="100" velocity="100"/>
     </joint>
     <joint name="horizontal_joint" type="prismatic">
@@ -47,13 +50,13 @@
       <parent link="vertical_link"/>
       <child link="horizontal_link"/>
-      <axis xyz="0.0 1.0 0.0"/>
+      <axis xyz="1.0 0.0 0.0"/>
       <limit upper="0.03" lower="-0.03" effort="100" velocity="100"/>
     </joint>
-    <joint name="vertical_joint" type="prismatic">
+    <joint name="insertion_joint" type="prismatic">
       <origin xyz="0 0 0" rpy="0 0 0"/>
-      <parent link="base_link"/>
-      <child link="vertical_link"/>
-      <axis xyz="0.0 0.0 1.0"/>
-      <limit upper="0.05" lower="0.0" effort="100" velocity="100"/>
+      <parent link="horizontal_link"/>
+      <child link="needle_link"/>
+      <axis xyz="0.0 1.0 0.0"/>
+      <limit upper="0.1" lower="0.0" effort="100" velocity="100"/>
     </joint>
   </xacro:macro>
