Commit message: Update galil_description with meshes. Create launch demo.launch for visualization testing

File: galil_description/urdf/galil.ros2_control.xacro (robot description, xacro)
@@ -9,9 +9,9 @@
         <command_interface name="position">
           <param name="min">0</param>
-          <param name="max">100</param>
+          <param name="max">0.1</param>
         </command_interface>
         <command_interface name="velocity">
-          <param name="min">-10</param>
-          <param name="max">10</param>
+          <param name="min">-0.005</param>
+          <param name="max"> 0.005</param>
         </command_interface>
         <state_interface name="position">
@@ -19,14 +19,13 @@
         </state_interface>
         <state_interface name="velocity"/>
-        <state_interface name="effort"/>
       </joint>
-      <joint name="template_horizontal_joint">
+      <joint name="horizontal_joint">
         <command_interface name="position">
-          <param name="min">0</param>
-          <param name="max">100</param>
+          <param name="min">-0.03</param>
+          <param name="max"> 0.03</param>
         </command_interface>
         <command_interface name="velocity">
-          <param name="min">-10</param>
-          <param name="max">10</param>
+          <param name="min">-0.005</param>
+          <param name="max"> 0.005</param>
         </command_interface>
         <state_interface name="position">
@@ -34,14 +33,13 @@
         </state_interface>
         <state_interface name="velocity"/>
-        <state_interface name="effort"/>
       </joint>
-      <joint name="template_vertical_joint">
+      <joint name="vertical_joint">
         <command_interface name="position">
-          <param name="min">0</param>
-          <param name="max">100</param>
+          <param name="min">   0</param>
+          <param name="max">0.05</param>
         </command_interface>
         <command_interface name="velocity">
-          <param name="min">-10</param>
-          <param name="max">10</param>
+          <param name="min">-0.005</param>
+          <param name="max"> 0.005</param>
         </command_interface>
         <state_interface name="position">
@@ -49,5 +47,4 @@
         </state_interface>
         <state_interface name="velocity"/>
-        <state_interface name="effort"/>
       </joint>
     </ros2_control>

File: galil_description/urdf/galil.xacro (robot description, xacro)
@@ -2,71 +2,58 @@
 <robot xmlns:xacro="http://wiki.ros.org/xacro">
   <xacro:macro name="galil">
-    <!-- links -  main serial chain -->
-    <link name="base_link"/>
-    <link name="insertion_link">
-      <visual>
-        <origin xyz="0 0 0" rpy="0 0 ${pi}"/>
-        <geometry>
-          <box size="1 1 1"/>
-	</geometry>
-      </visual>
-      <collision>
-        <origin xyz="0 0 0" rpy="0 0 ${pi}"/>
-        <geometry>
-          <box size="1 1 1"/>
-        </geometry>
-      </collision>
-    </link>
-    <joint name="insertion_joint" type="prismatic">
-      <origin xyz="0 0 0" rpy="0 0 0" />
-      <axis xyz="0 0 1" />
-      <parent link="base_link" />
-      <child link="insertion_link" />
-      <limit lower="0" upper="100"
-             effort="100" velocity="10"/>
-    </joint>
-    <link name="template_horizontal">
+    <xacro:include filename="$(find galil_description)/urdf/materials.xacro" />
+    <link name="base_link">
       <visual>
         <origin xyz="0 0 0" rpy="0 0 0"/>
         <geometry>
-          <box size="1 1 1"/>
-	</geometry>
+          <mesh filename="package://galil_description/meshes/base_link.stl"/>
+        </geometry>
+        <material name="silver"/>
       </visual>
-      <collision>
-        <origin xyz="0 0 0" rpy="0 0 0"/>
+    </link>
+    <link name="needle_link">
+      <visual>
         <geometry>
-          <box size="1 1 1"/>
+          <mesh filename="package://galil_description/meshes/needle_link.stl"/>
         </geometry>
-      </collision>
+        <material name="silver"/>
+      </visual>
     </link>
-    <joint name="template_horizontal_joint" type="prismatic">
-      <origin xyz="0 0 0" rpy="0 0 0" />
-      <axis xyz="0 0 1" />
-      <parent link="base_link" />
-      <child link="template_horizontal_link" />
-      <limit lower="0" upper="100"
-             effort="100" velocity="10"/>
+    <link name="vertical_link">
+      <visual>
+        <geometry>
+          <mesh filename="package://galil_description/meshes/vertical_link.stl"/>
+        </geometry>
+        <material name="silver"/>
+      </visual>
+    </link>
+    <link name="horizontal_link">
+      <visual>
+        <geometry>
+          <mesh filename="package://galil_description/meshes/horizontal_link.stl"/>
+        </geometry>
+        <material name="silver"/>
+      </visual>
+    </link>
+    <joint name="insertion_joint" type="prismatic">
+      <origin xyz="0 0 0" rpy="0 0 0"/>
+      <parent link="horizontal_link"/>
+      <child link="needle_link"/>
+      <axis xyz="-1.0 0.0 0.0"/>
+      <limit upper="0.1" lower="0.0" effort="100" velocity="100"/>
     </joint>
-    <link name="template_verticalal">
-      <visual>
-        <origin xyz="0 0 0" rpy="0 0 0"/>
-        <geometry>
-          <box size="1 1 1"/>
-	</geometry>
-      </visual>
-      <collision>
-        <origin xyz="0 0 0" rpy="0 0 0"/>
-        <geometry>
-          <box size="1 1 1"/>
-        </geometry>
-      </collision>
-    </link>
-    <joint name="template_vertical_joint" type="prismatic">
-      <origin xyz="0 0 0" rpy="0 0 0" />
-      <axis xyz="0 0 1" />
-      <parent link="template_horizontal_link" />
-      <child link="template_vertical_link" />
-      <limit lower="0" upper="100"
-             effort="100" velocity="10"/>
+    <joint name="horizontal_joint" type="prismatic">
+      <origin xyz="0 0 0" rpy="0 0 0"/>
+      <parent link="vertical_link"/>
+      <child link="horizontal_link"/>
+      <axis xyz="0.0 1.0 0.0"/>
+      <limit upper="0.03" lower="-0.03" effort="100" velocity="100"/>
+    </joint>
+    <joint name="vertical_joint" type="prismatic">
+      <origin xyz="0 0 0" rpy="0 0 0"/>
+      <parent link="base_link"/>
+      <child link="vertical_link"/>
+      <axis xyz="0.0 0.0 1.0"/>
+      <limit upper="0.05" lower="0.0" effort="100" velocity="100"/>
     </joint>
   </xacro:macro>

Commit message: update bwh, that will need to be removed to switch to PT

File: galil_description/urdf/galil.ros2_control.xacro (robot description, xacro)
@@ -6,8 +6,8 @@
         <plugin>galil_driver/GalilSystemHardwareInterface</plugin>
       </hardware>
-      <joint name="insertion_joint">
+      <joint name="horizontal_joint">
         <command_interface name="position">
-          <param name="min">0</param>
-          <param name="max">0.1</param>
+          <param name="min">-0.03</param>
+          <param name="max"> 0.03</param>
         </command_interface>
         <command_interface name="velocity">
@@ -20,8 +20,8 @@
         <state_interface name="velocity"/>
       </joint>
-      <joint name="horizontal_joint">
+      <joint name="insertion_joint">
         <command_interface name="position">
-          <param name="min">-0.03</param>
-          <param name="max"> 0.03</param>
+          <param name="min">0</param>
+          <param name="max">0.1</param>
         </command_interface>
         <command_interface name="velocity">
